File: pennyesc.kicad_pcb (KiCad board)
At the start: 4 copper layers, 15.9 x 14 mm, 28 parts, among them U1 STM32L011F4Ux, U2 MCT8316Z0RRGFR, U3 TMAG5273A1QDBVR

Commit message: add brushed firmware
Parts:
- R8: value 3.3k -> 1k
- U2: value MCT8316Z0RRGFR -> MCT8316Z0R
