File: pennyesc.kicad_sch (KiCad schematic)
At the start: 28 parts, among them U1 STM32L011F4Ux, U2 MCT8316Z0RRGFR, U3 TMAG5273A1QDBVR

Commit message: add brushed firmware
Parts:
- R2: value 1k -> 3.3k
- R8: value 3.3k -> 1k; JLCPCB C25890 -> C11702; LCSC PN C25890 -> C11702; MP 0402WGF3301TCE -> 0402WGF1001TCE
- U2: value MCT8316Z0RRGFR -> MCT8316Z0R; JLCPCB C3681249 -> C3681397; LCSC PN C3681249 -> C3681397; MP MCT8316Z0RRGFR -> MCT8316Z0RQRGFRQ1
Changed lines of the file:
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@@
 			)
 		)
-		(property "Value" "3.3k"
+		(property "Value" "1k"
 			(at 121.92 81.28 0)
 			(show_name no)
@@
 			)
 		)
-		(property "JLCPCB" "C25890"
+		(property "JLCPCB" "C11702"
 			(at 124.46 80.01 0)
 			(hide yes)
@@
 			)
 		)
-		(property "MP" "0402WGF3301TCE"
+		(property "MP" "0402WGF1001TCE"
 			(at 124.46 80.01 0)
 			(hide yes)
@@
 			)
 		)
-		(property "LCSC PN" "C25890"
+		(property "LCSC PN" "C11702"
 			(at 124.46 80.01 0)
 			(hide yes)
@@
 			)
 		)
-		(property "Value" "MCT8316Z0RRGFR"
+		(property "Value" "MCT8316Z0R"
 			(at 189.23 54.61 0)
 			(show_name no)
@@
 			)
 		)
-		(property "JLCPCB" "C3681249"
+		(property "JLCPCB" "C3681397"
 			(at 187.96 110.49 0)
 			(hide yes)
@@
 			)
 		)
-		(property "MP" "MCT8316Z0RRGFR"
+		(property "MP" "MCT8316Z0RQRGFRQ1"
 			(at 187.96 110.49 0)
 			(hide yes)
@@
 			)
 		)
-		(property "LCSC PN" "C3681249"
+		(property "LCSC PN" "C3681397"
 			(at 187.96 110.49 0)
 			(hide yes)
@@
 			)
 		)
-		(property "Value" "1k"
+		(property "Value" "3.3k"
 			(at 160.02 83.82 90)
 			(show_name no)
